Commit message: add zg m1 task and refine titatit collisions

File: assets/robots/titatit/urdf/wheeled_titatit_rl.urdf (robot description, URDF)
Before this commit: robot wheeled_titatit_description, 19 links, 18 joints
Links:
- link FL_calf: geometry collision box size=0.25 0.05 0.07; visual mesh filename=../dae/FL_calf.dae
- link FL_thigh: geometry collision box size=0.26 0.06 0.08; visual mesh filename=../dae/FL_thigh.dae
- link FR_calf: geometry collision box size=0.25 0.05 0.07; visual mesh filename=../dae/FR_calf.dae
- link FR_thigh: geometry collision box size=0.26 0.06 0.08; visual mesh filename=../dae/FR_thigh.dae
- link RL_calf: geometry collision box size=0.25 0.05 0.07; visual mesh filename=../dae/RL_calf.dae
- link RL_thigh: geometry collision box size=0.26 0.06 0.08; visual mesh filename=../dae/RL_thigh.dae
- link RR_calf: geometry collision box size=0.25 0.05 0.07; visual mesh filename=../dae/RR_calf.dae
- link RR_thigh: geometry collision box size=0.26 0.06 0.08; visual mesh filename=../dae/RR_thigh.dae
- link trunk: geometry collision box size=0.28 0.15 0.19; collision box size=0.28 0.15 0.19
